Commit message: [urdf]fix_v3_display_error

File: ranger_mini/ranger_mini_v2/urdf/ranger_mini.xacro (robot description, xacro)
@@ -20,5 +20,5 @@
             <origin xyz="0 0 0" rpy="1.57 0 3.14 " />
             <geometry>
-                <mesh filename="package://ranger_mini_v2/meshes/ranger_base.dae" />
+                <mesh filename="package://ranger_mini_v2/meshes/base_link.STL" />
             </geometry>
         </visual>
@@ -72,5 +72,5 @@
                 <origin xyz="0.23 -0.2 0.1" rpy="1.57 0 0" />
                 <geometry>
-                    <mesh filename="package://ranger_mini_v2/meshes/fr.dae" />
+                    <mesh filename="package://ranger_mini_v2/meshes/fr.stl" />
                 </geometry>
             </visual>
@@ -129,5 +129,5 @@
                 <origin xyz="0.23 0.2 0.1" rpy="1.57 0 0" />
                 <geometry>
-                    <mesh filename="package://ranger_mini_v2/meshes/fl.dae" />
+                    <mesh filename="package://ranger_mini_v2/meshes/fl.stl" />
                 </geometry>
             </visual>
@@ -186,5 +186,5 @@
                 <origin xyz="0.23 -0.2 0.1" rpy="1.57 0 0" />
                 <geometry>
-                    <mesh filename="package://ranger_mini_v2/meshes/fr.dae" />
+                    <mesh filename="package://ranger_mini_v2/meshes/fr.stl" />
                 </geometry>
             </visual>
@@ -243,5 +243,5 @@
                 <origin xyz="0.23 0.2 0.1" rpy="1.57 0 0" />
                 <geometry>
-                    <mesh filename="package://ranger_mini_v2/meshes/fl.dae" />
+                    <mesh filename="package://ranger_mini_v2/meshes/fl.stl" />
                 </geometry>
             </visual>
