Commit message: [urdf]ranegr_mini_v3_sensor_and_kinetics_model

File: ranger_mini/ranger_mini_v3/urdf/ranger_mini.xacro (robot description, xacro)
@@ -1,346 +1,326 @@
 <?xml version="1.0" encoding="utf-8"?>
-<robot name="ranger_mini_v3"  xmlns:xacro="http://ros.org/wiki/xacro">
-  <link
-    name="base_link">
-    <inertial>
-      <origin
-        xyz="-0.0242698272228022 -0.0030308024613212 0.0544267444673498"
-        rpy="0 0 0" />
-      <mass
-        value="10" />
+<robot name="ranger_mini_v3"
+  xmlns:xacro="http://ros.org/wiki/xacro">
+  <link name="base_footprint">
+    <visual>
+      <origin xyz="0 0 0" rpy="0 0 0"/>
+      <geometry>
+        <box size="0.001 0.001 0.001"/>
+      </geometry>
+    </visual>
+  </link>
+  <gazebo reference="base_footprint">
+    <turnGravityOff>false</turnGravityOff>
+  </gazebo>
+  <joint name="base_footprint_joint" type="fixed">
+    <origin xyz="0 0 0.30" rpy="0 0 0"/>
+    <parent link="base_footprint"/>
+    <child link="base_link"/>
+  </joint>
+  <link name="base_link">
+    <inertial>
+      <origin xyz="-0.0242698272228022 -0.0030308024613212 0.0544267444673498" rpy="0 0 0" />
+      <mass value="10" />
       <inertia ixx="0.1354" ixy="0.0" ixz="0.0" iyy="0.2417" iyz="0.0" izz="0.3085"/>
     </inertial>
     <visual>
-      <origin
-        xyz="0 0 0.0"
-        rpy="0 0 0" />
-      <geometry>
-        <mesh
-          filename="package://ranger_mini_v3/meshes/ranger_base.dae" scale="1000 1000 1000" />
-      </geometry>
-      <material
-        name="">
-        <color
-          rgba="0.792156862745098 0.819607843137255 0.933333333333333 1" />
+      <origin xyz="0 0 0.07" rpy="0 0 0" />
+      <geometry>
+        <mesh filename="package://ranger_mini_v3/meshes/ranger_base.dae" scale="1000 1000 1000" />
+      </geometry>
+      <material name="">
+        <color rgba="0.792156862745098 0.819607843137255 0.933333333333333 1" />
       </material>
     </visual>
-        <collision>
-            <origin xyz="0 0 -0.1" rpy="0 0 0" />
-            <geometry>
-                <box size="0.5 0.35 0.2"/>
-            </geometry>
-        </collision>
-   </link>
-   <link
-    name="fr_steering_wheel_link">
-    <inertial>
-      <origin
-        xyz="1.8493E-05 1.2713E-06 0.043679"
-        rpy="0 0 0" />
-      <mass
-        value="1" />
-      <inertia
-        ixx="0.0063625"
-        ixy="-1.0581E-07"
-        ixz="-4.0831E-07"
-        iyy="0.006363"
-        iyz="-3.4944E-08"
-        izz="0.010465" />
-    </inertial>
-    <visual>
-      <origin
-        xyz="0 0 0"
-        rpy="0 0 0" />
+    <collision>
+      <origin xyz="0 0 0" rpy="0 0 0" />
+      <geometry>
+        <box size="0.72 0.5 0.14"/>
+      </geometry>
+    </collision>
+  </link>
+  <link name="fr_steering_wheel_link">
+    <inertial>
+      <origin xyz="1.8493E-05 1.2713E-06 0.043679" rpy="0 0 0" />
+      <mass value="1" />
+      <inertia ixx="0.0063625" ixy="-1.0581E-07" ixz="-4.0831E-07" iyy="0.006363" iyz="-3.4944E-08" izz="0.010465" />
+    </inertial>
+    <visual>
+      <origin xyz="0 0 0" rpy="0 0 0" />
       <geometry>
         <mesh filename="package://ranger_mini_v3/meshes/steering_wheel.dae" scale="10 10 10"/>
       </geometry>
-      <material
-        name="">
-        <color
-          rgba="0.79216 0.81961 0.93333 1" />
+      <material name="">
+        <color rgba="0.79216 0.81961 0.93333 1" />
       </material>
     </visual>
     <collision>
-      <origin
-        xyz="0 0 0"
-        rpy="0 0 0" />
-      <geometry>
-        <!-- <mesh
-          filename="package://ranger_mini_v3/meshes/ranger_mini_v3_wheel_right.dae" /> -->
-          <cylinder radius="0.001" length="0.001"/>
-      </geometry>
-    </collision>
-  </link>
-  <joint
-    name="fr_steering_joint"
-    type="revolute">
-    <origin
-      xyz="0.25 -0.19 -0.1"
-      rpy="0 0 0" />
-    <parent
-      link="base_link" />
-    <child
-      link="fr_steering_wheel_link" />
-    <axis
-      xyz="0 0 -1" />
-    <limit effort="5" velocity="6.28"  lower="-2.1" upper="2.1" />
+      <origin xyz="0 0 0" rpy="0 0 0" />
+      <geometry>
+        <!-- <mesh filename="package://ranger_mini_v3/meshes/ranger_mini_v3_wheel_right.dae" /> -->
+        <cylinder radius="0.001" length="0.001"/>
+      </geometry>
+    </collision>
+  </link>
+  <joint name="fr_steering_joint" type="revolute">
+    <origin xyz="0.25 -0.19 -0.07" rpy="0 0 0" />
+    <parent link="base_link" />
+    <child link="fr_steering_wheel_link" />
+    <axis xyz="0 0 -1" />
+    <limit effort="5" velocity="6.28" lower="-2.1" upper="2.1" />
   </joint>
   <link name="fr_wheel_link">
-      <inertial>
-          <mass value="8" />
-          <origin xyz="0 0 0" />
-          <inertia ixx="0.02047" ixy="0.0" ixz="0.0" iyy="0.02047" iyz="0.0" izz="0.0324"/>
-          </inertial>
-      <visual>
-          <origin xyz="0 0 0" rpy="3.14 0 0" />
-          <geometry>
-            <mesh filename="package://ranger_mini_v3/meshes/wheel_v3.dae" scale="10 10 10"/>
-          </geometry>
-      </visual>
-      <collision>
-          <origin xyz="0 0 -0.005" rpy="1.57 0 0" />
-          <geometry>
-              <cylinder length="0.08" radius="0.09" />
-          </geometry>
-                <contact>
-                    <ode>
-                  <min_depth>0.001</min_depth>
-                    </ode>
-              </contact>
-      </collision>
-  </link>
-        <joint name="fr_wheel" type="continuous">
-            <origin xyz="0.0 0.0 -0.12" rpy="0 0 0" />
-            <parent link="fr_steering_wheel_link"/>
-            <child link="fr_wheel_link"/>
-            <axis xyz="0 1 0" rpy="0 0 0" />
-        </joint>
-  <link
-    name="fl_steering_wheel_link">
-    <inertial>
-      <origin
-        xyz="-0.0017956 -9.6304E-08 0.043642"
-        rpy="0 0 0" />
-      <mass
-        value="1" />
-      <inertia
-        ixx="0.0063695"
-        ixy="-2.1067E-08"
-        ixz="-0.00016867"
-        iyy="0.006363"
-        iyz="-1.0301E-08"
-        izz="0.010458" />
-    </inertial>
-    <visual>
-      <origin
-        xyz="0 0 0"
-        rpy="0 0 3.14" />
+    <inertial>
+      <mass value="8" />
+      <origin xyz="0 0 0" />
+      <inertia ixx="0.02047" ixy="0.0" ixz="0.0" iyy="0.02047" iyz="0.0" izz="0.0324"/>
+    </inertial>
+    <visual>
+      <origin xyz="0 0 0" rpy="3.14 0 0" />
+      <geometry>
+        <mesh filename="package://ranger_mini_v3/meshes/wheel_v3.dae" scale="10 10 10"/>
+      </geometry>
+    </visual>
+    <collision>
+      <origin xyz="0 0 -0.005" rpy="1.57 0 0" />
+      <geometry>
+        <cylinder length="0.08" radius="0.09" />
+      </geometry>
+      <contact>
+        <ode>
+          <min_depth>0.001</min_depth>
+        </ode>
+      </contact>
+    </collision>
+  </link>
+  <joint name="fr_wheel" type="continuous">
+    <origin xyz="0.0 0.0 -0.12" rpy="0 0 0" />
+    <parent link="fr_steering_wheel_link"/>
+    <child link="fr_wheel_link"/>
+    <axis xyz="0 1 0" rpy="0 0 0" />
+  </joint>
+  <link name="fl_steering_wheel_link">
+    <inertial>
+      <origin xyz="-0.0017956 -9.6304E-08 0.043642" rpy="0 0 0" />
+      <mass value="1" />
+      <inertia ixx="0.0063695" ixy="-2.1067E-08" ixz="-0.00016867" iyy="0.006363" iyz="-1.0301E-08" izz="0.010458" />
+    </inertial>
+    <visual>
+      <origin xyz="0 0 0" rpy="0 0 3.14" />
       <geometry>
         <mesh filename="package://ranger_mini_v3/meshes/steering_wheel.dae" scale="10 10 10"/>
       </geometry>
-      <material
-        name="">
-        <color
-          rgba="0.79216 0.81961 0.93333 1" />
+      <material name="">
+        <color rgba="0.79216 0.81961 0.93333 1" />
       </material>
     </visual>
     <collision>
-      <origin
-        xyz="0 0 0"
-        rpy="0 0 0" />
-      <geometry>
-        <!-- <mesh
-          filename="package://ranger_mini_v3/meshes/ranger_mini_v3_wheel.dae" /> -->
+      <origin xyz="0 0 0" rpy="0 0 0" />
+      <geometry>
+        <!-- <mesh filename="package://ranger_mini_v3/meshes/ranger_mini_v3_wheel.dae" /> -->
         <cylinder radius="0.001" length="0.001"/>
       </geometry>
     </collision>
   </link>
-   <joint
-    name="fl_steering_joint"
-    type="revolute">
-    <origin
-      xyz="0.25 0.19 -0.1"
-      rpy="0 0 0" />
-    <parent
-      link="base_link" />
-    <child
-      link="fl_steering_wheel_link" />
-    <axis
-      xyz="0 0 -1" />
-        <limit effort="5" velocity="6.28"  lower="-2.1" upper="2.1" />
-  </joint>
-        <link name="fl_wheel_link">
-            <inertial>
-                <mass value="8" />
-                <origin xyz="0 0 0" />
-                <inertia ixx="0.02047" ixy="0.0" ixz="0.0" iyy="0.02047" iyz="0.0" izz="0.0324"/>
-            </inertial>
-            <visual>
-                <origin xyz="0 0 0" rpy="0 0 0" />
-                <geometry>
-                <mesh filename="package://ranger_mini_v3/meshes/wheel_v3.dae" scale="10 10 10"/>
-                </geometry>
-            </visual>
-            <collision>
-                <origin xyz="0 0 -0.005" rpy="1.57 0 0" />
-                <geometry>
-                    <cylinder length="0.08" radius="0.09" />
-                </geometry>
-                     <contact>
-                         <ode>
-                        <min_depth>0.001</min_depth>
-                         </ode>
-                    </contact>
-            </collision>
-        </link>
-        <joint name="fl_wheel" type="continuous">
-            <origin xyz="0.0 0.0 -0.12" rpy="0 0 0" />
-            <parent link="fl_steering_wheel_link"/>
-            <child link="fl_wheel_link"/>
-            <axis xyz="0 1 0" rpy="0 0 0" />
-        </joint>
- <link
-    name="rl_steering_wheel_link">
-    <inertial>
-      <origin
-        xyz="-0.00017093 6.1255E-08 0.043678"
-        rpy="0 0 0" />
-      <mass
-        value="1" />
-      <inertia
-        ixx="0.0063627"
-        ixy="-2.1069E-08"
-        ixz="-1.587E-05"
-        iyy="0.006363"
-        iyz="9.3201E-09"
-        izz="0.010465" />
-    </inertial>
-    <visual>
-      <origin
-        xyz="0 0 0"
-        rpy="0 0 3.14" />
+  <joint name="fl_steering_joint" type="revolute">
+    <origin xyz="0.25 0.19 -0.07" rpy="0 0 0" />
+    <parent link="base_link" />
+    <child link="fl_steering_wheel_link" />
+    <axis xyz="0 0 -1" />
+    <limit effort="5" velocity="6.28" lower="-2.1" upper="2.1" />
+  </joint>
+  <link name="fl_wheel_link">
+    <inertial>
+      <mass value="8" />
+      <origin xyz="0 0 0" />
+      <inertia ixx="0.02047" ixy="0.0" ixz="0.0" iyy="0.02047" iyz="0.0" izz="0.0324"/>
+    </inertial>
+    <visual>
+      <origin xyz="0 0 0" rpy="0 0 0" />
+      <geometry>
+        <mesh filename="package://ranger_mini_v3/meshes/wheel_v3.dae" scale="10 10 10"/>
+      </geometry>
+    </visual>
+    <collision>
+      <origin xyz="0 0 -0.005" rpy="1.57 0 0" />
+      <geometry>
+        <cylinder length="0.08" radius="0.09" />
+      </geometry>
+      <contact>
+        <ode>
+          <min_depth>0.001</min_depth>
+        </ode>
+      </contact>
+    </collision>
+  </link>
+  <joint name="fl_wheel" type="continuous">
+    <origin xyz="0.0 0.0 -0.12" rpy="0 0 0" />
+    <parent link="fl_steering_wheel_link"/>
+    <child link="fl_wheel_link"/>
+    <axis xyz="0 1 0" rpy="0 0 0" />
+  </joint>
+  <link name="rl_steering_wheel_link">
+    <inertial>
+      <origin xyz="-0.00017093 6.1255E-08 0.043678" rpy="0 0 0" />
+      <mass value="1" />
+      <inertia ixx="0.0063627" ixy="-2.1069E-08" ixz="-1.587E-05" iyy="0.006363" iyz="9.3201E-09" izz="0.010465" />
+    </inertial>
+    <visual>
+      <origin xyz="0 0 0" rpy="0 0 3.14" />
       <geometry>
         <mesh filename="package://ranger_mini_v3/meshes/steering_wheel.dae" scale="10 10 10"/>
       </geometry>
-      <material
-        name="">
-        <color
-          rgba="0.79216 0.81961 0.93333 1" />
+      <material name="">
+        <color rgba="0.79216 0.81961 0.93333 1" />
       </material>
     </visual>
     <collision>
-      <origin
-        xyz="0 0 0"
-        rpy="0 0 0" />
-      <geometry>
-        <!-- <mesh
-          filename="package://ranger_mini_v3/meshes/ranger_mini_v3_wheel_right.dae" /> -->
+      <origin xyz="0 0 0" rpy="0 0 0" />
+      <geometry>
+        <!-- <mesh filename="package://ranger_mini_v3/meshes/ranger_mini_v3_wheel_right.dae" /> -->
         <cylinder radius="0.001" length="0.001"/>
       </geometry>
     </collision>
   </link>
-  <joint
-    name="rl_steering_joint"
-    type="revolute">
-    <origin
-      xyz="-0.25 0.19 -0.1"
-      rpy="0 0 0" />
-    <parent
-      link="base_link" />
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
Commit message: [rviz]validate_controller_for_ranger_and_add_a_sim_environment

File: ranger_mini/ranger_mini_v3/urdf/ranger_mini.xacro (robot description, xacro)
@@ -87,9 +87,19 @@
         <cylinder length="0.08" radius="0.09" />
       </geometry>
-      <contact>
-        <ode>
-          <min_depth>0.001</min_depth>
-        </ode>
-      </contact>
+      <surface>
+        <friction>
+          <ode>
+            <mu>5.0</mu>
+            <mu2>5.0</mu2>
+          </ode>
+        </friction>
+        <contact>
+          <ode>
+            <slip1>0.001</slip1>
+            <slip2>0.001</slip2>
+            <min_depth>0.001</min_depth>
+          </ode>
+        </contact>
+      </surface>
     </collision>
   </link>
@@ -147,9 +157,19 @@
         <cylinder length="0.08" radius="0.09" />
       </geometry>
-      <contact>
-        <ode>
-          <min_depth>0.001</min_depth>
-        </ode>
-      </contact>
+      <surface>
+        <friction>
+          <ode>
+            <mu>5.0</mu>
+            <mu2>5.0</mu2>
+          </ode>
+        </friction>
+        <contact>
+          <ode>
+            <slip1>0.001</slip1>
+            <slip2>0.001</slip2>
+            <min_depth>0.001</min_depth>
+          </ode>
+        </contact>
+      </surface>
     </collision>
   </link>
@@ -207,9 +227,19 @@
         <cylinder length="0.08" radius="0.09" />
       </geometry>
-      <contact>
-        <ode>
-          <min_depth>0.001</min_depth>
-        </ode>
-      </contact>
+      <surface>
+        <friction>
+          <ode>
+            <mu>5.0</mu>
+            <mu2>5.0</mu2>
+          </ode>
+        </friction>
+        <contact>
+          <ode>
+            <slip1>0.001</slip1>
+            <slip2>0.001</slip2>
+            <min_depth>0.001</min_depth>
+          </ode>
+        </contact>
+      </surface>
     </collision>
   </link>
@@ -263,9 +293,19 @@
         <cylinder length="0.08" radius="0.09" />
       </geometry>
-      <contact>
-        <ode>
-          <min_depth>0.001</min_depth>
-        </ode>
-      </contact>
+      <surface>
+        <friction>
+          <ode>
+            <mu>5.0</mu>
+            <mu2>5.0</mu2>
+          </ode>
+        </friction>
+        <contact>
+          <ode>
+            <slip1>0.001</slip1>
+            <slip2>0.001</slip2>
+            <min_depth>0.001</min_depth>
+          </ode>
+        </contact>
+      </surface>
     </collision>
   </link>
@@ -322,88 +362,87 @@
   <xacro:include filename="$(find ranger_mini_v3)/urdf/sensor/laser.xacro" />
   <xacro:laser joint_x="${laser_joint_x}" joint_y="${laser_joint_y}" joint_z="${laser_joint_z}" parent_link="laser_stand_link"/>
-  <!--
-	<transmission name="fl_steering_wheel_trans">
-      <type>transmission_interface/SimpleTransmission</type>
-      <joint name="fl_steering_joint">
-		<hardwareInterface>hardware_interface/PositionJointInterface</hardwareInterface>
-      </joint>
-	  <actuator name="fl_steering_wheel_motor">
-		<hardwareInterface>hardware_interface/PositionJointInterface</hardwareInterface>
-		<mechanicalReduction>30</mechanicalReduction>
-      </actuator>
-	</transmission>
-	<transmission name="fr_steering_wheel_trans">
-      <type>transmission_interface/SimpleTransmission</type>
-      <joint name="fr_steering_joint">
-		<hardwareInterface>hardware_interface/PositionJointInterface</hardwareInterface>
-      </joint>
-	  <actuator name="fr_steering_wheel_motor">
-		<hardwareInterface>hardware_interface/PositionJointInterface</hardwareInterface>
-		<mechanicalReduction>30</mechanicalReduction>
-      </actuator>
-	</transmission>
-	<transmission name="rl_steering_wheel_trans">
-      <type>transmission_interface/SimpleTransmission</type>
-      <joint name="rl_steering_joint">
-		<hardwareInterface>hardware_interface/PositionJointInterface</hardwareInterface>
-      </joint>
-	  <actuator name="rl_steering_wheel_motor">
-		<hardwareInterface>hardware_interface/PositionJointInterface</hardwareInterface>
-		<mechanicalReduction>30</mechanicalReduction>
-      </actuator>
-	</transmission>
-	<transmission name="rr_steering_wheel_trans">
-      <type>transmission_interface/SimpleTransmission</type>
-      <joint name="rr_steering_joint">
-		<hardwareInterface>hardware_interface/PositionJointInterface</hardwareInterface>
-      </joint>
-	  <actuator name="rr_steering_wheel_motor">
-		<hardwareInterface>hardware_interface/PositionJointInterface</hardwareInterface>
-		<mechanicalReduction>30</mechanicalReduction>
-      </actuator>
-	</transmission>
-	<transmission name="fl_wheel_trans">
-      <type>transmission_interface/SimpleTransmission</type>
-      <joint name="fl_wheel">
-		<hardwareInterface>hardware_interface/VelocityJointInterface</hardwareInterface>
-      </joint>
-	  <actuator name="fl_wheel_motor">
-		<hardwareInterface>hardware_interface/VelocityJointInterface</hardwareInterface>
-		<mechanicalReduction>30</mechanicalReduction>
-      </actuator>
-	</transmission>
-	<transmission name="fr_wheel_trans">
-      <type>transmission_interface/SimpleTransmission</type>
-      <joint name="fr_wheel">
-		<hardwareInterface>hardware_interface/VelocityJointInterface</hardwareInterface>
-      </joint>
-	  <actuator name="fr_wheel_motor">
-		<hardwareInterface>hardware_interface/VelocityJointInterface</hardwareInterface>
-		<mechanicalReduction>30</mechanicalReduction>
-      </actuator>
-	</transmission>
-	<transmission name="rl_wheel_trans">
-      <type>transmission_interface/SimpleTransmission</type>
-      <joint name="rl_wheel">
-		<hardwareInterface>hardware_interface/VelocityJointInterface</hardwareInterface>
-      </joint>
-	  <actuator name="rl_wheel_motor">
-		<hardwareInterface>hardware_interface/VelocityJointInterface</hardwareInterface>
-		<mechanicalReduction>30</mechanicalReduction>
-      </actuator>
-	</transmission>
-	<transmission name="rr_wheel_trans">
-      <type>transmission_interface/SimpleTransmission</type>
-      <joint name="rr_wheel">
-		<hardwareInterface>hardware_interface/VelocityJointInterface</hardwareInterface>
-      </joint>
-	  <actuator name="rr_wheel_motor">
-		<hardwareInterface>hardware_interface/VelocityJointInterface</hardwareInterface>
-		<mechanicalReduction>30</mechanicalReduction>
-      </actuator>
-	</transmission>
+  <transmission name="fl_steering_wheel_trans">
+    <type>transmission_interface/SimpleTransmission</type>
+    <joint name="fl_steering_joint">
+      <hardwareInterface>hardware_interface/PositionJointInterface</hardwareInterface>
+    </joint>
+    <actuator name="fl_steering_wheel_motor">
+      <hardwareInterface>hardware_interface/PositionJointInterface</hardwareInterface>
+      <mechanicalReduction>30</mechanicalReduction>
+    </actuator>
+  </transmission>
+  <transmission name="fr_steering_wheel_trans">
+    <type>transmission_interface/SimpleTransmission</type>
+    <joint name="fr_steering_joint">
+      <hardwareInterface>hardware_interface/PositionJointInterface</hardwareInterface>
+    </joint>
+    <actuator name="fr_steering_wheel_motor">
+      <hardwareInterface>hardware_interface/PositionJointInterface</hardwareInterface>
+      <mechanicalReduction>30</mechanicalReduction>
+    </actuator>
+  </transmission>
+  <transmission name="rl_steering_wheel_trans">
+    <type>transmission_interface/SimpleTransmission</type>
+    <joint name="rl_steering_joint">
+      <hardwareInterface>hardware_interface/PositionJointInterface</hardwareInterface>
+    </joint>
+    <actuator name="rl_steering_wheel_motor">
+      <hardwareInterface>hardware_interface/PositionJointInterface</hardwareInterface>
+      <mechanicalReduction>30</mechanicalReduction>
+    </actuator>
+  </transmission>
+  <transmission name="rr_steering_wheel_trans">
+    <type>transmission_interface/SimpleTransmission</type>
+    <joint name="rr_steering_joint">
+      <hardwareInterface>hardware_interface/PositionJointInterface</hardwareInterface>
+    </joint>
+    <actuator name="rr_steering_wheel_motor">
+      <hardwareInterface>hardware_interface/PositionJointInterface</hardwareInterface>
+      <mechanicalReduction>30</mechanicalReduction>
+    </actuator>
+  </transmission>
+  <transmission name="fl_wheel_trans">
+    <type>transmission_interface/SimpleTransmission</type>
+    <joint name="fl_wheel">
+      <hardwareInterface>hardware_interface/VelocityJointInterface</hardwareInterface>
+    </joint>
+    <actuator name="fl_wheel_motor">
+      <hardwareInterface>hardware_interface/VelocityJointInterface</hardwareInterface>
+      <mechanicalReduction>30</mechanicalReduction>
+    </actuator>
+  </transmission>
+  <transmission name="fr_wheel_trans">
+    <type>transmission_interface/SimpleTransmission</type>
+    <joint name="fr_wheel">
+      <hardwareInterface>hardware_interface/VelocityJointInterface</hardwareInterface>
+    </joint>
+    <actuator name="fr_wheel_motor">
+      <hardwareInterface>hardware_interface/VelocityJointInterface</hardwareInterface>
+      <mechanicalReduction>30</mechanicalReduction>
+    </actuator>
+  </transmission>
+  <transmission name="rl_wheel_trans">
+    <type>transmission_interface/SimpleTransmission</type>
+    <joint name="rl_wheel">
+      <hardwareInterface>hardware_interface/VelocityJointInterface</hardwareInterface>
+    </joint>
+    <actuator name="rl_wheel_motor">
+      <hardwareInterface>hardware_interface/VelocityJointInterface</hardwareInterface>
+      <mechanicalReduction>30</mechanicalReduction>
+    </actuator>
+  </transmission>
+  <transmission name="rr_wheel_trans">
+    <type>transmission_interface/SimpleTransmission</type>
+    <joint name="rr_wheel">
+      <hardwareInterface>hardware_interface/VelocityJointInterface</hardwareInterface>
+    </joint>
+    <actuator name="rr_wheel_motor">
+      <hardwareInterface>hardware_interface/VelocityJointInterface</hardwareInterface>
+      <mechanicalReduction>30</mechanicalReduction>
+    </actuator>
+  </transmission>
   <gazebo>
     <plugin name="gazebo_ros_control" filename="libgazebo_ros_control.so">
     </plugin>
-  </gazebo> -->
+  </gazebo>
 </robot>
