Commit message: [navigation]ranger_v3_navigation_uncompleted

File: ranger_mini/ranger_mini_v3/urdf/ranger_mini.xacro (robot description, xacro)
@@ -67,5 +67,5 @@
     <parent link="base_link" />
     <child link="fr_steering_wheel_link" />
-    <axis xyz="0 0 -1" />
+    <axis xyz="0 0 1" />
     <limit effort="5" velocity="6.28" lower="-2.1" upper="2.1" />
   </joint>
@@ -137,5 +137,5 @@
     <parent link="base_link" />
     <child link="fl_steering_wheel_link" />
-    <axis xyz="0 0 -1" />
+    <axis xyz="0 0 1" />
     <limit effort="5" velocity="6.28" lower="-2.1" upper="2.1" />
   </joint>
@@ -207,5 +207,5 @@
     <parent link="base_link" />
     <child link="rl_steering_wheel_link" />
-    <axis xyz="0 0 -1" />
+    <axis xyz="0 0 1" />
     <limit effort="5" velocity="6.28" lower="-2.1" upper="2.1" />
   </joint>
@@ -273,5 +273,5 @@
     <parent link="base_link"/>
     <child link="rr_steering_wheel_link"/>
-    <axis xyz="0 0 -1" rpy="0 0 0" />
+    <axis xyz="0 0 1" rpy="0 0 0" />
     <limit effort="5" velocity="6.28" lower="-2.1" upper="2.1" />
   </joint>

File: ranger_mini/ranger_mini_v3/urdf/sensor/laser.xacro (robot description, xacro)
@@ -37,17 +37,17 @@
         <pose>0 0 0 0 0 0</pose>
         <visualize>false</visualize>
-        <update_rate>5.5</update_rate>
+        <update_rate>15.0</update_rate>
         <ray>
           <scan>
             <horizontal>
-              <samples>360</samples>
+              <samples>720</samples>
               <resolution>1</resolution>
-              <min_angle>-3</min_angle>
-              <max_angle>3</max_angle>
+              <min_angle>-3.1415926</min_angle>
+              <max_angle>3.1415926</max_angle>
             </horizontal>
           </scan>
           <range>
             <min>0.10</min>
-            <max>6.0</max>
+            <max>25.0</max>
             <resolution>0.01</resolution>
           </range>

Commit message: better_navigation and dynamic avoidance test

File: ranger_mini/ranger_mini_v3/urdf/ranger_mini.xacro (robot description, xacro)
@@ -355,4 +355,7 @@
   <xacro:property name="laser_joint_y" value="0.0" />
   <xacro:property name="laser_joint_z" value="0.08" />
+  <xacro:property name="imu_joint_x" value="0.0" />
+  <xacro:property name="imu_joint_y" value="0.0" />
+  <xacro:property name="imu_joint_z" value="0.12" />
   <!-- 传感器集成 -->
   <xacro:include filename="$(find ranger_mini_v3)/urdf/sensor/camera.xacro" />
@@ -362,4 +365,6 @@
   <xacro:include filename="$(find ranger_mini_v3)/urdf/sensor/laser.xacro" />
   <xacro:laser joint_x="${laser_joint_x}" joint_y="${laser_joint_y}" joint_z="${laser_joint_z}" parent_link="laser_stand_link"/>
+  <xacro:include filename="$(find ranger_mini_v3)/urdf/sensor/imu.xacro" />
+  <xacro:imu joint_x="${imu_joint_x}" joint_y="${imu_joint_y}" joint_z="${imu_joint_z}" parent_link="base_link"/>
   <transmission name="fl_steering_wheel_trans">
     <type>transmission_interface/SimpleTransmission</type>

File: ranger_mini/ranger_mini_v3/urdf/sensor/laser.xacro (robot description, xacro)
@@ -36,5 +36,5 @@
       <sensor type="gpu_ray" name="rplidar">
         <pose>0 0 0 0 0 0</pose>
-        <visualize>true</visualize>
+        <visualize>false</visualize>
         <update_rate>15.0</update_rate>
         <ray>
